Commit message: Update (Unsaved).xacro

File: urdf/(Unsaved)_description/urdf/(Unsaved).xacro (robot description, xacro)
@@ -94,5 +94,5 @@
   <parent link="base_link"/>
   <child link="whell_1"/>
-  <axis xyz="-0.0 -1.0 -0.0"/>
+  <axis xyz="0.0 1.0 0.0"/>
 </joint>
 <joint name="Rigid6" type="fixed">
